Commit message: Testing

File: ariac_description/urdf/ariac_robots/ariac_robots.urdf.xacro (robot description, xacro)
@@ -16,5 +16,4 @@
   <xacro:include filename="$(find ariac_description)/urdf/floor_robot/floor_robot_macro.xacro"/>
   <xacro:include filename="$(find ariac_description)/urdf/ceiling_robot/ceiling_robot_macro.xacro"/>
-  <xacro:include filename="$(find ariac_description)/urdf/agv/agv_macro.xacro"/>
   <!-- Define arguments for robot cameras -->
   <xacro:arg name="floor_robot_camera_active_arg" default="false"/>
@@ -36,28 +35,8 @@
     camera_type="${ceiling_robot_camera_type}">
   </xacro:ceiling_robot>
-  <!-- AGV1 -->
-  <xacro:agv
-    agv_number="agv1"
-    y_position="4.8" >
-  </xacro:agv>
-  <!-- AGV2 -->
-  <xacro:agv
-    agv_number="agv2"
-    y_position="1.2" >
-  </xacro:agv>
-  <!-- AGV3 -->
-  <xacro:agv
-    agv_number="agv3"
-    y_position="-1.2" >
-  </xacro:agv>
-  <!-- AGV4 -->
-  <xacro:agv
-    agv_number="agv4"
-    y_position="-4.8" >
-  </xacro:agv>
   <gazebo
     reference="world">
   </gazebo>
-  <!-- ROS2 Control Plugin -->
+  <!-- ROS2 Control Plugin -->Z
   <xacro:arg name="controllers" default="$(find ariac_description)/config/robot_controllers.yaml" />
   <gazebo>

File: ariac_description/urdf/ceiling_robot/ceiling_robot_macro.xacro (robot description, xacro)
@@ -5,29 +5,22 @@
     camera_type
   ">
-    <xacro:include filename="$(find ariac_description)/urdf/ceiling_robot/gantry_macro.xacro"/>
+    <!-- Include linear actuator macro -->
+    <xacro:include filename="$(find ariac_description)/urdf/ceiling_robot/linear_actuator_macro_2.xacro"/>
     <!-- Inclue ur robot macro -->
-    <xacro:include filename="$(find ur_description)/urdf/ur_macro.xacro"/>
+    <xacro:include filename="$(find franka_description)/robots/panda_arm.xacro"/>
     <!-- Inclue gripper macro -->
-    <xacro:include filename="$(find ariac_description)/urdf/vacuum_gripper/vacuum_gripper_macro.xacro"/>
+    <xacro:include filename="$(find franka_description)/robots/hand.xacro"/>
     <xacro:property name="initial_positions_file" default="$(find ariac_description)/config/ceiling_robot_initial_positions.yaml"/>
-    <!-- Run gantry macro -->
-    <xacro:gantry
+    <!-- Run linear actuator macro -->
+    <xacro:linear_actuator_2
       parent="world"
-      long_rail_length="15.0"
-      long_rail_width="0.2"
-      long_rail_offset="-5.0"
-      small_rail_length="15.0"
-      small_rail_width="0.2"
-      rail_height="2.9"
-      rail_thickness="0.1"
-      torso_height="-2.3"
       initial_positions="${xacro.load_yaml(initial_positions_file)}"
       >
-    </xacro:gantry>
+    </xacro:linear_actuator_2>
     <!-- Run ur macro -->
-    <xacro:ur_robot
-      name="ceiling_arm"
-      tf_prefix="ceiling_"
-      parent="torso_main"
+    <xacro:panda_arm
+      name="panda_arm"
+      tf_prefix="floor_"
+      parent="robot_base"
       joint_limits_parameters_file="$(find ur_description)/config/ur10e/joint_limits.yaml"
       kinematics_parameters_file="$(find ur_description)/config/ur10e/default_kinematics.yaml"
@@ -36,15 +29,12 @@
       sim_gazebo="true"
       initial_positions="${xacro.load_yaml(initial_positions_file)}">
-      <origin xyz="0.51 0.0 1.3" rpy="0 1.57 0" />
-    </xacro:ur_robot>
+      <origin xyz="0 0 0.05" rpy="0 0 0" />
+    </xacro:panda_arm>
     <!-- Run gripper macro -->
-    <xacro:vacuum_gripper
-      parent="wrist_3_link"
-      prefix="ceiling"
-      use_camera="${camera_active}"
-      camera_type="${camera_type}"
-      >
-    </xacro:vacuum_gripper>
-    <xacro:arg name="controllers" default="$(find ariac_description)/config/robot_controllers.yaml" />
+    <xacro:hand
+    ns="panda"
+    rpy="0 0 ${-pi/4}"
+    connected_to="panda_link8"
+    safety_distance="0.0"/>
   </xacro:macro>
 </robot>

File: ariac_description/urdf/floor_robot/linear_actuator_macro.xacro (robot description, xacro)
@@ -13,5 +13,5 @@
       <visual>
         <geometry>
-          <box size="0.2 10 0.1"/>
+          <box size="0.2 0.1 0.1"/>
         </geometry>
         <origin xyz="0 0 0"/>
@@ -20,5 +20,5 @@
       <collision>
         <geometry>
-          <box size="0.2 10 0.1"/>
+          <box size="0.2 0.1 0.1"/>
         </geometry>
       </collision>
@@ -40,5 +40,5 @@
       <parent link="${parent}"/>
       <child link="slide_bar"/>
-      <origin xyz="-1.3 0.0 0.93" rpy="0.0 0.0 ${pi}"/>
+      <origin xyz="0.2 3.0 0.8" rpy="0.0 0.0 1.57"/>
     </joint>
     <joint name="linear_actuator_joint" type="prismatic">

Commit message: Spawns two robots!!!

File: ariac_description/urdf/ariac_robots/ariac_robots.urdf.xacro (robot description, xacro)
@@ -15,5 +15,5 @@
   <!-- Locate Robot Macros -->
   <xacro:include filename="$(find ariac_description)/urdf/floor_robot/floor_robot_macro.xacro"/>
-  <xacro:include filename="$(find ariac_description)/urdf/ceiling_robot/ceiling_robot_macro.xacro"/>
+  <xacro:include filename="$(find ariac_description)/urdf/second_floor_robot/floor_robot_2_macro.xacro"/>
   <!-- Define arguments for robot cameras -->
   <xacro:arg name="floor_robot_camera_active_arg" default="false"/>
@@ -30,9 +30,8 @@
     camera_type="${floor_robot_camera_type}">
   </xacro:floor_robot>
-  <!-- Ceiling Robot -->
-  <xacro:ceiling_robot
+  <xacro:floor_robot_2
     camera_active="${ceiling_robot_camera_active}"
     camera_type="${ceiling_robot_camera_type}">
-  </xacro:ceiling_robot>
+  </xacro:floor_robot_2>
   <gazebo
     reference="world">

File: ariac_description/urdf/floor_robot/linear_actuator_macro.xacro (robot description, xacro)
@@ -40,5 +40,5 @@
       <parent link="${parent}"/>
       <child link="slide_bar"/>
-      <origin xyz="0.2 3.0 0.8" rpy="0.0 0.0 1.57"/>
+      <origin xyz="0.2 -3.0 0.8" rpy="0.0 0.0 1.57"/>
     </joint>
     <joint name="linear_actuator_joint" type="prismatic">
