Commit message: Trying to get bins to work

File: ariac_description/urdf/floor_robot/linear_actuator_macro.xacro (robot description, xacro)
@@ -40,5 +40,5 @@
       <parent link="${parent}"/>
       <child link="slide_bar"/>
-      <origin xyz="0.2 -3.0 0.8" rpy="0.0 0.0 1.57"/>
+      <origin xyz="0.5 -3.0 0.8" rpy="0.0 0.0 1.57"/>
     </joint>
     <joint name="linear_actuator_joint" type="prismatic">

File: ariac_description/urdf/second_floor_robot/floor_robot_2_macro.xacro (robot description, xacro)
@@ -33,5 +33,5 @@
       sim_gazebo="true"
       initial_positions="${xacro.load_yaml(initial_positions_file)}">
-      <origin xyz="7.0 0.0 0.0" rpy="0.0 0.0 ${pi}"/>
+      <origin xyz="6.5 0.25 0.0" rpy="0.0 0.0 ${pi}"/>
     </xacro:ur_robot>
     <!-- Run gripper macro -->
